File: Hardware/KiCad/RP2040_WEDS.kicad_pcb (KiCad board)
At the start: 2 copper layers, 55 x 66 mm, 75 parts, among them J1 Barrel_Jack_Switch_Pin3Ring, J2 Analog Soil Header, J3 LiPo Batt, J4 I2C Soil Header, J5 Conn_02x05_Odd_Even, J6 SMA-J-P-H-RA-TH1, J7 USB Header, Q1 Q_PMOS_DGS, Q2 Q_PMOS_DGS, SW1 SW_Push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

Commit message: Updated filepaths
Parts:
- U1: footprint RP2040KICAD:QFN40P700X700X90-57N -> 54-00125:QFN40P700X700X90-57N
- renumbered USB to J8

Commit message: Adjusted copper fill
Routing:
- net +BATT: track 22.5 -> 6.98 mm
- net VDD: track 27.9 -> 15.7 mm
- net GND: track 137.1 -> 127.3 mm, vias 46 -> 44
