File: Hardware/KiCad/RP2040_WEDS-backups/RP2040_WEDS-2022-02-14_145055/RP2040_WEDS.kicad_sch (KiCad schematic)
At the start: 75 parts, among them J1 Barrel_Jack_Switch_Pin3Ring, J2 Conn_01x02_Male, J3 I2C Soil Header, J4 LiPo Batt, J5 Analog Soil Header, J6 USB Header, J7 Conn_02x05_Odd_Even, J8 SMA-J-P-H-RA-TH1, Q1 Q_PMOS_DGS, Q2 Q_PMOS_DGS, SW1 SW_Push, SW2 SW_Push, SW3 SW_Push, U1 RP2040, U2 MCP73831-2-OT, U3 W25Q128JVS, U4 BME280, U5 AP2112K-3.3, U6 LoRa-E5, U7 TPL5110, Y1 Crystal_GND24

Commit message: changes
Parts:
- removed J2: Conn_01x02_Male, Connector_PinHeader_1.27mm:PinHeader_1x02_P1.27mm_Vertical, symbol Connector:Conn_01x02_Male
- removed R6: 1k, Resistor_SMD:R_0603_1608Metric, symbol Device:R
- C15: renamed from C16; value 100nF -> C
- U1: footprint 54-00125:QFN40P700X700X90-57N -> RP2040KICAD:QFN40P700X700X90-57N
- renumbered C12 to C11, C13 to C12, C14 to C13, C15 to C14, C17 to C16, C18 to C17, C19 to C18, C20 to C19, C21 to C20, C22 to C21, C23 to C22, C24 to C23, C9 to C24, C11 to C9, J5 to J2, J4 to J3, J3 to J4, J7 to J5, J8 to J6, J6 to J7, R2 to R1, R13 to R10, R14 to R11, R15 to R12, R16 to R13, R17 to R14, R3 to R15, R4 to R16, R1 to R2, R5 to R3, R7 to R4, R8 to R5, R9 to R6, R10 to R7, R11 to R8, R12 to R9, TP3 to TP1, TP4 to TP2, TP1 to TP3, TP2 to TP4
Connections:
- no-connect marks 41 -> 22
Other:
- note added: "Power Isolation"
